File: aviyonik/aviyonik.kicad_pcb (KiCad board)
At the start: 4 copper layers, 69.8 x 71.5 mm, 125 parts, among them J1 Conn_01x06_Pin, J10 Conn_01x03_Pin, J11 Conn_01x03_Pin, J12 Screw_Terminal_01x02, J2 Screw_Terminal_01x02, J3 Conn_01x03_Pin, J4 Screw_Terminal_01x02, J5 Conn_01x03_Pin, J6 Conn_01x03_Pin, J7 Conn_01x03_Pin, J8 USB_C_Receptacle_USB2.0_16P, J9 MEM2061-01-188-00-A, SW1 SW_SPDT, U10 MCP1700x-120xxMB, U11 USBLC6-2P6, U12 ISM330IS, U2 MS5611-01BA, U3 MMC5983MA, U4 ICM-42686-P, U5 SCH16T-K01-10, U6 STM32H755ZITx, U7 TCAN1044VDRQ1, U8 TCAN1044VDRQ1, U9 INA226AIDGST, Y1 XO32

Commit message: F.cu ground pour has been added and iamges changed
Routing:
- net GND: vias 124 -> 147

Commit message: revision
connectors have been revisioned
3.3 to 1.8 ldo's have been added to imu's
5 to 3.3v ldo have been changed
i2c and uart connectors have been added for gps and pitot tube connections
Parts:
- removed C53: 10uF, Capacitor_THT:CP_Radial_D4.0mm_P2.00mm
- removed U10: MCP1700x-120xxMB, Package_TO_SOT_SMD:SOT-89-3
- added C59: 1u, Capacitor_SMD:C_0805_2012Metric_Pad1.18x1.45mm_HandSolder, F.Cu at (171.7, 54.0)
- added C60: 1u, Capacitor_SMD:C_0805_2012Metric_Pad1.18x1.45mm_HandSolder, F.Cu at (171.6, 61.4)
- added C61: 1u, Capacitor_SMD:C_0805_2012Metric_Pad1.18x1.45mm_HandSolder, F.Cu at (148.2, 114.2)
- added C62: 1u, Capacitor_SMD:C_0805_2012Metric_Pad1.18x1.45mm_HandSolder, F.Cu at (151.7, 111.0)
- added J13: Conn_01x04_Pin, Connector_JST:JST_GH_SM04B-GHS-TB_1x04-1MP_P1.25mm_Horizontal, F.Cu at (175.9, 117.9)
- added U1: LP5907MFX-1.8, Package_TO_SOT_SMD:SOT-23-5, F.Cu at (171.8, 57.2)
- added U13: LP5907MFX-1.8, Package_TO_SOT_SMD:SOT-23-5, F.Cu at (151.6, 114.1)
- added U14: LD1117S33TR_SOT223, Package_TO_SOT_SMD:SOT-223-3_TabPin2, F.Cu at (187.6, 98.4)
- C52: value 1uF -> 4.7u
- J10: value Conn_01x03_Pin -> Conn_01x06_Pin; footprint Connector_PinHeader_2.54mm:PinHeader_1x03_P2.54mm_Vertical -> Connector_JST:JST_GH_SM06B-GHS-TB_1x06-1MP_P1.25mm_Horizontal
- J12: footprint Connector_PinHeader_2.54mm:PinHeader_1x02_P2.54mm_Vertical_SMD_Pin1Left -> Connector_Wire:SolderWire-0.5sqmm_1x02_P4.6mm_D0.9mm_OD2.1mm
- J2, J4: value Screw_Terminal_01x02 -> Conn_01x04_Pin; footprint Connector_PinHeader_2.00mm:PinHeader_1x02_P2.00mm_Vertical -> Connector_JST:JST_GH_SM04B-GHS-TB_1x04-1MP_P1.25mm_Horizontal
- R27: footprint Resistor_SMD:R_0805_2012Metric_Pad1.20x1.40mm_HandSolder -> Resistor_SMD:R_2512_6332Metric
- moved R21 22.1 mm to (203.8, 105.1), turned to -90 degrees
- moved R20 19.1 mm to (201.6, 105.1), turned to -90 degrees
- moved D4 16.7 mm to (203.8, 109.3), turned to -90 degrees
- moved R19 16.4 mm to (199.3, 105.1), turned to -90 degrees
- moved D3 14.1 mm to (201.6, 109.3), turned to -90 degrees
- moved D2 12.2 mm to (199.3, 109.4), turned to -90 degrees
- moved R27 10.6 mm to (187.2, 108.8), turned to 0 degrees
- moved C46 10.5 mm to (201.6, 113.3), turned to -90 degrees
- moved J2 10.2 mm to (185.8, 118.0), turned to 0 degrees
- moved C52 4.39 mm to (186.1, 103.2), turned to 0 degrees
- moved J10 4.28 mm to (158.8, 118.2), turned to 0 degrees
- moved J11 3.72 mm to (150.3, 119.8)
- moved C55 3.24 mm to (198.0, 85.1)
- moved U7 3.01 mm to (187.2, 56.9), turned to -90 degrees
- moved R33 2.97 mm to (200.2, 61.0)
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Connections:
- net /MCU/AP_CS renamed /FLIGHT CONTROLLER/AP_CS
- net /MCU/AP_INT renamed /FLIGHT CONTROLLER/AP_INT
- net /MCU/AP_MISO renamed /FLIGHT CONTROLLER/AP_MISO
- net /MCU/AP_MOSI renamed /FLIGHT CONTROLLER/AP_MOSI
- net /MCU/AP_SCK renamed /FLIGHT CONTROLLER/AP_SCK
- net /MCU/BAR_SCL renamed /FLIGHT CONTROLLER/BAR_SCL
- net /MCU/BAR_SDA renamed /FLIGHT CONTROLLER/BAR_SDA
- net /MCU/BLUE renamed /FLIGHT CONTROLLER/BLUE
- net /MCU/CAN1H renamed /FLIGHT CONTROLLER/CAN1H
- net /MCU/CAN2H renamed /FLIGHT CONTROLLER/CAN2H
- net /MCU/CUR_ALERT renamed /FLIGHT CONTROLLER/CUR_ALERT
- net /MCU/DRY_SYNC renamed /FLIGHT CONTROLLER/DRY_SYNC
- net /MCU/EXTRESN renamed /FLIGHT CONTROLLER/EXTRESN
- net /MCU/GREEN renamed /FLIGHT CONTROLLER/GREEN
- net /MCU/IMU_CS renamed /FLIGHT CONTROLLER/IMU_CS
- net /MCU/IMU_INT renamed /FLIGHT CONTROLLER/IMU_INT
- net /MCU/IMU_MISO renamed /FLIGHT CONTROLLER/IMU_MISO
- net /MCU/IMU_MOSI renamed /FLIGHT CONTROLLER/IMU_MOSI
- net /MCU/IMU_SCK renamed /FLIGHT CONTROLLER/IMU_SCK
- net /MCU/MAG_INT renamed /FLIGHT CONTROLLER/MAG_INT
- net /MCU/RED renamed /FLIGHT CONTROLLER/RED
- net /MCU/SCH_CS renamed /FLIGHT CONTROLLER/SCH_CS
- net /MCU/SCH_MISO renamed /FLIGHT CONTROLLER/SCH_MISO
- net /MCU/SCH_MOSI renamed /FLIGHT CONTROLLER/SCH_MOSI
- net /MCU/SCH_SCK renamed /FLIGHT CONTROLLER/SCH_SCK
- net /MCU/SD_CLK renamed /FLIGHT CONTROLLER/SD_CLK
- net /MCU/SD_CMD renamed /FLIGHT CONTROLLER/SD_CMD
- net /MCU/SD_DAT0 renamed /FLIGHT CONTROLLER/SD_DAT0
- net /MCU/SD_DAT1 renamed /FLIGHT CONTROLLER/SD_DAT1
- net /MCU/SD_DAT2 renamed /FLIGHT CONTROLLER/SD_DAT2
- net /MCU/SD_DAT3 renamed /FLIGHT CONTROLLER/SD_DAT3
- net /MCU/SD_NCD renamed /FLIGHT CONTROLLER/SD_NCD
- net /MCU/USB_DN renamed /FLIGHT CONTROLLER/USB_DN
- net /MCU/USB_DP renamed /FLIGHT CONTROLLER/USB_DP
- C1 pad 1: +3.3V -> +1V8
- C10 pad 1: +3.3V -> +1V8
- C2 pad 1: +3.3V -> +1V8
- C55 pad 1: Net-(C55-Pad1) -> Net-(J12-Pin_1)
- C56 pad 1: Net-(C55-Pad1) -> Net-(J12-Pin_1)
- C9 pad 1: +3.3V -> +1V8
- F1 pad 1: Net-(C55-Pad1) -> Net-(J12-Pin_1)
- FB2 pad 2: Net-(C55-Pad1) -> Net-(J12-Pin_1)
- J10 pad 1: USART2_RX -> +5V
- J10 pad 3: GND -> USART2_RX
- J12 pad 1: +5V -> Net-(J12-Pin_1)
- J2 pad 1: /MCU/CAN2L -> +5V
- J4 pad 1: /MCU/CAN1L -> +5V
- R5 pad 1: /MCU/CUR_SDA -> I2C_SDA
- R6 pad 2: /MCU/CUR_SCL -> I2C_SCL
- R7 pad 2: +3.3V -> +1V8
- U12 pad 8: +3.3V -> +1V8
- U3 pad 1: /MCU/CUR_SCL -> I2C_SCL
- U3 pad 16: /MCU/CUR_SDA -> I2C_SDA
- U6 pad 123: unconnected-(U6-PG10-Pad123) -> /FLIGHT CONTROLLER/ICM_EN
- U6 pad 48: unconnected-(U6-PC5-Pad48) -> /FLIGHT CONTROLLER/ISM_EN
- U6 pad 66: /MCU/CUR_SCL -> I2C_SCL
- U6 pad 67: /MCU/CUR_SDA -> I2C_SDA
- U7 pad 6: /MCU/CAN1L -> /FLIGHT CONTROLLER/CAN1L
- U8 pad 6: /MCU/CAN2L -> /FLIGHT CONTROLLER/CAN2L
- U9 pad 4: /MCU/CUR_SDA -> I2C_SDA
- U9 pad 5: /MCU/CUR_SCL -> I2C_SCL
Routing:
- net I2C_SCL: track 0.00 -> 65.3 mm, vias 0 -> 6
- net I2C_SDA: track 0.00 -> 60.2 mm, vias 0 -> 3
- net +5V: track 129.4 -> 165.4 mm, vias 17 -> 13
- net /FLIGHT CONTROLLER/ISM_EN: track 0.00 -> 31.5 mm, vias 0 -> 2
- net RGB_R: track 28.8 -> 58.0 mm
- net /MCU/CUR_SCL: track 28.2 -> 0.00 mm, vias 2 -> 0
- net /MCU/CUR_SDA: track 26.3 -> 0.00 mm
- net /FLIGHT CONTROLLER/ICM_EN: track 0.00 -> 21.2 mm, vias 0 -> 2
- net /Power/R_SHUNT+: track 30.1 -> 15.3 mm
- net RGB_B: track 22.1 -> 35.5 mm
- net RGB_G: track 22.7 -> 34.8 mm
- net /FLIGHT CONTROLLER/CAN2H: track 11.2 -> 22.1 mm
- net /FLIGHT CONTROLLER/CAN2L: track 0.00 -> 10.7 mm
- net /FLIGHT CONTROLLER/CAN1L: track 0.00 -> 10.6 mm
- net /MCU/CAN2L: track 8.91 -> 0.00 mm
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- added copper zone on F.Cu, net +1V8
- added copper zone on In2.Cu, net +1V8
- added copper zone on F.Cu, net /Power/R_SHUNT+
- added copper zone on F.Cu, net Net-(J12-Pin_1)
- added copper zone on In2.Cu, net Net-(J12-Pin_1)
- removed copper zone on F.Cu, net Net-(C55-Pad1)
- removed copper zone on In2.Cu, net Net-(C55-Pad1)
Other:
- outline, holes or cut-outs redrawn
- board text added: "5V"
- board text added: "GND"

Commit message: revision
3.3 to 1.8 LDO's added to IMU Voltage Input
5 to 3.3 LDO have been revisioned
I2C and UART headers have been added for GPS and Pitot Tube connections
5V and GND pins have been corrected
Connections:
- C1 pad 1: +1V8 -> ISM_VDD(1V8)
- C10 pad 1: +1V8 -> ICM_VDD(1V8)
- C2 pad 1: +1V8 -> ISM_VDD(1V8)
- C60 pad 1: +1V8 -> ICM_VDD(1V8)
- C62 pad 1: +1V8 -> ISM_VDD(1V8)
- C9 pad 1: +1V8 -> ICM_VDD(1V8)
- R7 pad 2: +1V8 -> ICM_VDD(1V8)
- U1 pad 5: +1V8 -> ICM_VDD(1V8)
- U12 pad 8: +1V8 -> ISM_VDD(1V8)
- U13 pad 5: +1V8 -> ISM_VDD(1V8)
Routing:
- net ISM_VDD(1V8): track 0.00 -> 4.13 mm, vias 0 -> 4
- net +1V8: track 4.13 -> 0.00 mm, vias 4 -> 0
- added copper zone on F.Cu, net ICM_VDD(1V8)
- added copper zone on F.Cu, net ISM_VDD(1V8)
- added copper zone on In2.Cu, net ISM_VDD(1V8)
- removed copper zone on F.Cu, net +1V8
- removed copper zone on In2.Cu, net +1V8
Changed lines of the file:
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@@
 			(layers "F.Cu" "F.Mask" "F.Paste")
 			(roundrect_rratio 0.212766)
-			(net "+1V8")
+			(net "ICM_VDD(1V8)")
 			(pintype "passive")
 		)
@@
 			(layers "F.Cu" "F.Mask" "F.Paste")
 			(roundrect_rratio 0.25)
-			(net "+1V8")
+			(net "ISM_VDD(1V8)")
 			(pinfunction "VDD_8")
 			(pintype "power_in")
@@
 			(layers "F.Cu" "F.Mask" "F.Paste")
 			(roundrect_rratio 0.212766)
-			(net "+1V8")
+			(net "ISM_VDD(1V8)")
 			(pintype "passive")
 		)
@@
 			(layers "F.Cu" "F.Mask" "F.Paste")
 			(roundrect_rratio 0.208333)
-			(net "+1V8")
+			(net "ICM_VDD(1V8)")
 			(pintype "passive")
 		)
@@
 			(layers "F.Cu" "F.Mask" "F.Paste")
 			(roundrect_rratio 0.212766)
-			(net "+1V8")
+			(net "ISM_VDD(1V8)")
 			(pintype "passive")
 		)
@@
 			(layers "F.Cu" "F.Mask" "F.Paste")
 			(roundrect_rratio 0.212766)
-			(net "+1V8")
+			(net "ICM_VDD(1V8)")
 			(pintype "passive")
 		)
@@
 			(layers "F.Cu" "F.Mask" "F.Paste")
 			(roundrect_rratio 0.25)
-			(net "+1V8")
+			(net "ISM_VDD(1V8)")
 			(pinfunction "OUT_5")
 			(pintype "power_out")
@@
 			(layers "F.Cu" "F.Mask" "F.Paste")
 			(roundrect_rratio 0.25)
-			(net "+1V8")
+			(net "ICM_VDD(1V8)")
 			(pinfunction "OUT_5")
 			(pintype "power_out")
@@
 			(layers "F.Cu" "F.Mask" "F.Paste")
 			(roundrect_rratio 0.212766)
-			(net "+1V8")
+			(net "ICM_VDD(1V8)")
 			(pintype "passive")
 		)
@@
 			(layers "F.Cu" "F.Mask" "F.Paste")
 			(roundrect_rratio 0.212766)
-			(net "+1V8")
+			(net "ISM_VDD(1V8)")
 			(pintype "passive")
 		)
@@
 	)
 	(segment
-		(start 156.6875 109.95)
-		(end 156.6875 112.125)
-		(width 0.8)
-		(layer "F.Cu")
-		(net "+1V8")
-	)
-	(segment
-		(start 158.5375 109.7)
-		(end 156.9375 109.7)
-		(width 0.2)
-		(layer "F.Cu")
-		(net "+1V8")
-	)
-	(segment
-		(start 156.9375 109.7)
-		(end 156.6875 109.95)
-		(width 0.2)
-		(layer "F.Cu")
-		(net "+1V8")
-	)
-	(via
-		(at 152.43 109.51)
-		(size 0.6)
-		(drill 0.3)
-		(layers "F.Cu" "B.Cu")
-		(free yes)
-		(net "+1V8")
-	)
-	(via
-		(at 153.24 109.51)
-		(size 0.6)
-		(drill 0.3)
-		(layers "F.Cu" "B.Cu")
-		(free yes)
-		(net "+1V8")
-	)
-	(via
-		(at 157.54 108.43)
-		(size 0.6)
-		(drill 0.3)
-		(layers "F.Cu" "B.Cu")
-		(free yes)
-		(net "+1V8")
-	)
-	(via
-		(at 156.78 108.2)
-		(size 0.6)
-		(drill 0.3)
-		(layers "F.Cu" "B.Cu")
-		(free yes)
-		(net "+1V8")
-	)
-	(segment
 		(start 175.69 81.05559)
 		(end 175.69 81.17)
@@
 		(net "Net-(U4-AP_CS)")
 	)
+	(segment
+		(start 156.6875 109.95)
+		(end 156.6875 112.125)
+		(width 0.8)
+		(layer "F.Cu")
+		(net "ISM_VDD(1V8)")
+	)
+	(segment
+		(start 158.5375 109.7)
+		(end 156.9375 109.7)
+		(width 0.2)
+		(layer "F.Cu")
+		(net "ISM_VDD(1V8)")
+	)
+	(segment
+		(start 156.9375 109.7)
+		(end 156.6875 109.95)
+		(width 0.2)
+		(layer "F.Cu")
+		(net "ISM_VDD(1V8)")
+	)
+	(via
+		(at 152.43 109.51)
+		(size 0.6)
+		(drill 0.3)
+		(layers "F.Cu" "B.Cu")
+		(free yes)
+		(net "ISM_VDD(1V8)")
+	)
+	(via
+		(at 153.24 109.51)
+		(size 0.6)
+		(drill 0.3)
+		(layers "F.Cu" "B.Cu")
+		(free yes)
+		(net "ISM_VDD(1V8)")
+	)
+	(via
+		(at 157.54 108.43)
+		(size 0.6)
+		(drill 0.3)
+		(layers "F.Cu" "B.Cu")
+		(free yes)
+		(net "ISM_VDD(1V8)")
+	)
+	(via
+		(at 156.78 108.2)
+		(size 0.6)
+		(drill 0.3)
+		(layers "F.Cu" "B.Cu")
+		(free yes)
+		(net "ISM_VDD(1V8)")
+	)
 	(zone
 		(net "+3.3V")
@@
 	)
 	(zone
-		(net "+1V8")
+		(net "ISM_VDD(1V8)")
 		(layer "F.Cu")
 		(name "1V8")
@@
 	)
 	(zone
-		(net "+1V8")
+		(net "ISM_VDD(1V8)")
 		(layer "F.Cu")
 		(name "1V8")
@@
 	)
 	(zone
-		(net "+1V8")
+		(net "ICM_VDD(1V8)")
 		(layer "F.Cu")
 		(name "1V8")
@@
 	)
 	(zone
-		(net "+1V8")
+		(net "ISM_VDD(1V8)")
 		(layer "In2.Cu")
 		(name "1V8")
