File: aviyonik/aviyonik.kicad_pcb (KiCad board)
At the start: 4 copper layers, 69.8 x 71.5 mm, 140 parts, among them J10 Conn_01x06_Pin, J11 Conn_01x03_Pin, J12 Screw_Terminal_01x02, J13 Conn_01x04_Pin, J14 Conn_01x05, J2 Conn_01x04_Pin, J3 Conn_01x03_Pin, J4 Conn_01x04_Pin, J5 Conn_01x03_Pin, J6 Conn_01x03_Pin, J7 Conn_01x03_Pin, J8 USB_C_Receptacle_USB2.0_16P, J9 MEM2061-01-188-00-A, SW1 SW_SPDT, U1 LP5907MFX-1.8, U11 USBLC6-2P6, U12 ISM330IS, U13 LP5907MFX-1.8, U14 LD1117S33TR_SOT223, U2 MS5611-01BA, U3 MMC5983MA, U4 ICM-42686-P, U5 SCH16T-K01-10, U6 STM32H755ZITx, U7 TCAN1044VDRQ1, U8 TCAN1044VDRQ1, U9 INA226AIDGST, Y1 XO32

Commit message: power rails have been revised
Parts:
- removed J11, J5, J6, J7: Conn_01x03_Pin, Connector_PinHeader_2.54mm:PinHeader_1x03_P2.54mm_Vertical
- removed R15, R16, R17, R18: 33, Resistor_SMD:R_0805_2012Metric_Pad1.20x1.40mm_HandSolder
- added J1: Conn_01x04_Pin, Connector_JST:JST_GH_SM04B-GHS-TB_1x04-1MP_P1.25mm_Horizontal, F.Cu at (140.8, 110.9)
- J3: value Conn_01x03_Pin -> Conn_01x06; footprint Connector_PinHeader_2.54mm:PinHeader_1x03_P2.54mm_Vertical -> Connector_JST:JST_GH_SM06B-GHS-TB_1x06-1MP_P1.25mm_Horizontal
- moved F1 15.4 mm to (195.8, 96.6)
- moved J3 12.7 mm to (140.8, 99.7), turned to -90 degrees
- moved R25 9.89 mm to (194.7, 86.6), turned to -90 degrees
- moved R24 9.67 mm to (194.3, 92.7)
- moved FB2 7.84 mm to (202.6, 99.1), turned to 0 degrees
- moved C54 7.64 mm to (198.5, 99.7), turned to -90 degrees
- moved C56 1.03 mm to (195.6, 80.4), turned to 0 degrees
- moved C19 0.88 mm to (181.2, 84.1)
- moved C38 0.88 mm to (181.2, 88.5)
- moved C39 0.88 mm to (181.2, 86.3)
- moved C55 0.70 mm to (198.6, 85.2)
Connections:
- C54 pad 1: /Power/5V_GIRIS -> Net-(C54-Pad1)
- C55 pad 1: Net-(J12-Pin_1) -> +5V
- C56 pad 1: Net-(J12-Pin_1) -> +5V
- F1 pad 1: Net-(J12-Pin_1) -> /Power/5V_GIRIS
- F1 pad 2: +5V -> Net-(C54-Pad1)
- FB2 pad 1: /Power/5V_GIRIS -> Net-(C54-Pad1)
- FB2 pad 2: Net-(J12-Pin_1) -> +5V
- J12 pad 1: Net-(J12-Pin_1) -> +5V
- J3 pad 1: +3.3V -> GND
- J3 pad 2: PWM1 -> PGOOD_MAIN
- J3 pad 3: GND -> V_BAK
- U6 pad 28: unconnected-(U6-PC0-Pad28) -> V_BAK
- U6 pad 49: unconnected-(U6-PB0-Pad49) -> ST
- U6 pad 50: unconnected-(U6-PB1-Pad50) -> PGOOD_MAIN
- U6 pad 52: unconnected-(U6-PF11-Pad52) -> 5V_CRIT
- U6 pad 59: Net-(U6-PE9) -> unconnected-(U6-PE9-Pad59)
- U6 pad 61: Net-(U6-PE11) -> unconnected-(U6-PE11-Pad61)
- U6 pad 63: Net-(U6-PE13) -> unconnected-(U6-PE13-Pad63)
- U6 pad 64: Net-(U6-PE14) -> unconnected-(U6-PE14-Pad64)
- U6 pad 72: CAN2_TX -> CAN2_RX
- U6 pad 73: CAN2_RX -> CAN2_TX
Routing:
- net ST: track 0.00 -> 30.0 mm, vias 0 -> 2
- net Net-(U6-PE14): track 29.7 -> 0.00 mm, vias 2 -> 0
- net PGOOD_MAIN: track 0.00 -> 27.3 mm, vias 0 -> 2
- net 5V_CRIT: track 0.00 -> 26.7 mm, vias 0 -> 2
- net Net-(U6-PE13): track 26.2 -> 0.00 mm, vias 2 -> 0
- net Net-(U6-PE11): track 23.3 -> 0.00 mm, vias 2 -> 0
- net V_BAK: track 0.00 -> 21.5 mm, vias 0 -> 2
- net Net-(U6-PE9): track 20.3 -> 0.00 mm, vias 2 -> 0
- net PWM1: track 15.7 -> 0.00 mm
- net +5V: track 181.4 -> 196.6 mm, vias 13 -> 23
- net Net-(J8-CC1): track 17.3 -> 3.45 mm, vias 2 -> 0
- net GND: track 286.0 -> 273.4 mm, vias 223 -> 241
- net PWM2: track 12.4 -> 0.00 mm
- net PWM3: track 10.6 -> 0.00 mm
- net Net-(J8-CC2): track 16.0 -> 5.43 mm, vias 2 -> 0
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- added copper zone on F.Cu, net Net-(C54-Pad1)
- removed copper zone on F.Cu, net Net-(J12-Pin_1)
- removed copper zone on In2.Cu, net Net-(J12-Pin_1)
Other:
- board text removed: "5V"
- board text removed: "GND"
