File: aviyonik/sensors.kicad_sch (KiCad schematic)
At the start: 33 parts, among them U12 ISM330IS, U2 MS5611-01BA, U3 MMC5983MA, U4 ICM-42686-P, U5 SCH16T-K01-10, U9 INA226AIDGST

Commit message: revision
connectors have been revisioned
3.3 to 1.8 ldo's have been added to imu's
5 to 3.3v ldo have been changed
i2c and uart connectors have been added for gps and pitot tube connections
Parts:
- added C59, C60, C61, C62: 1u, Capacitor_SMD:C_0805_2012Metric_Pad1.18x1.45mm_HandSolder, symbol Device:C
- added U1, U13: LP5907MFX-1.8, Package_TO_SOT_SMD:SOT-23-5, symbol Regulator_Linear:LP5907MFX-1.8
Connections:
- net +3.3V: now also C59.1, C61.1, U1.1 (IN), U13.1 (IN); no longer C1.1, C10.1, C2.1, C9.1, R7.2, U12.8 (VDD)
- net GND: now also C59.2, C60.2, C61.2, C62.2, U1.2 (GND), U13.2 (GND)
- new net +1V8: C1.1, C10.1, C2.1, C60.1, C62.1, C9.1, R7.2, U1.5 (OUT), U12.8 (VDD), U13.5 (OUT)
- new net ICM_EN: U1.3 (EN)
- new net ISM_EN: U13.3 (EN)

Commit message: revision
3.3 to 1.8 LDO's added to IMU Voltage Input
5 to 3.3 LDO have been revisioned
I2C and UART headers have been added for GPS and Pitot Tube connections
5V and GND pins have been corrected
Connections:
- net +1V8 renamed ICM_VDD(1V8)
- net ICM_VDD(1V8): no longer C1.1, C2.1, C62.1, U12.8 (VDD), U13.5 (OUT)
- new net ISM_VDD(1V8): C1.1, C2.1, C62.1, U12.8 (VDD), U13.5 (OUT)
Changed lines of the file:
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@@
 			)
 		)
-		(property "Value" "+1V8"
-			(at 266.7 127 0)
+		(property "Value" "ICM_VDD(1V8)"
+			(at 269.24 130.8099 0)
 			(show_name no)
 			(do_not_autoplace no)
@@
 					(size 1.27 1.27)
 				)
+				(justify left)
 			)
 		)
@@
 			)
 		)
-		(property "Value" "+1V8"
-			(at 243.84 231.14 0)
+		(property "Value" "ISM_VDD(1V8)"
+			(at 246.38 234.9499 0)
 			(show_name no)
 			(do_not_autoplace no)
@@
 					(size 1.27 1.27)
 				)
+				(justify left)
 			)
 		)
@@
 		(in_pos_files yes)
 		(dnp no)
-		(fields_autoplaced yes)
 		(property "Reference" "#PWR02"
 			(at 78.74 30.48 0)
@@
 			)
 		)
-		(property "Value" "+1V8"
-			(at 78.74 21.59 0)
+		(property "Value" "ISM_VDD(1V8)"
+			(at 64.262 25.146 0)
 			(show_name no)
 			(do_not_autoplace no)
@@
 					(size 1.27 1.27)
 				)
+				(justify left)
 			)
 		)
@@
 			)
 		)
-		(property "Value" "+1V8"
-			(at 243.84 199.39 0)
+		(property "Value" "ICM_VDD(1V8)"
+			(at 246.38 203.1999 0)
 			(show_name no)
 			(do_not_autoplace no)
@@
 					(size 1.27 1.27)
 				)
+				(justify left)
 			)
 		)

Commit message: schematic changes
Connections:
- net +3.3V: now also U3.13 (VDDIO), U3.2 (VDD), U3.4 (~{SPI_CS})
- net AP_MISO: now also R10.1; no longer R9.1
- net AP_MOSI: now also R9.1; no longer R10.1
- net GND: now also C6.2, C7.1, U5.5 (RESERVED), U5.7 (RESERVED)
- no-connect marks 7 -> 5
Other:
- moved on the sheet: C6, C7
