File: aviyonik/mcu.kicad_sch (KiCad schematic)
At the start: 66 parts, among them J1 Conn_01x06_Pin, J10 Conn_01x03_Pin, J11 Conn_01x03_Pin, J12 Screw_Terminal_01x02, J2 Screw_Terminal_01x02, J3 Conn_01x03_Pin, J4 Screw_Terminal_01x02, J5 Conn_01x03_Pin, J6 Conn_01x03_Pin, J7 Conn_01x03_Pin, SW1 SW_SPDT, U6 STM32H755ZITx, U7 TCAN1044VDRQ1, U8 TCAN1044VDRQ1, Y1 XO32

Commit message: revision
connectors have been revisioned
3.3 to 1.8 ldo's have been added to imu's
5 to 3.3v ldo have been changed
i2c and uart connectors have been added for gps and pitot tube connections
Parts:
- removed J10: Conn_01x03_Pin, Connector_PinHeader_2.54mm:PinHeader_1x03_P2.54mm_Vertical, symbol Connector:Conn_01x03_Pin
- removed J12: Screw_Terminal_01x02, Connector_PinHeader_2.54mm:PinHeader_1x02_P2.54mm_Vertical_SMD_Pin1Left, symbol Connector:Screw_Terminal_01x02
- removed J2, J4: Screw_Terminal_01x02, Connector_PinHeader_2.00mm:PinHeader_1x02_P2.00mm_Vertical, symbol Connector:Screw_Terminal_01x02
- added J10: Conn_01x06_Pin, Connector_JST:JST_GH_SM06B-GHS-TB_1x06-1MP_P1.25mm_Horizontal, symbol Connector:Conn_01x06_Pin
- added J13, J2, J4: Conn_01x04_Pin, Connector_JST:JST_GH_SM04B-GHS-TB_1x04-1MP_P1.25mm_Horizontal, symbol Connector:Conn_01x04_Pin
Connections:
- net +5V: now also J10.1 (Pin_1), J13.1 (Pin_1), J2.1 (Pin_1), J4.1 (Pin_1)
- net CAN1H: now also J4.2 (Pin_2)
- net CAN1L: now also J4.3 (Pin_3)
- net CAN2H: now also J2.2 (Pin_2)
- net CAN2L: now also J2.3 (Pin_3)
- net GND: now also J10.6 (Pin_6), J13.4 (Pin_4), J2.4 (Pin_4), J4.4 (Pin_4)
- net USART2_RX: now also J10.3 (Pin_3)
- net USART2_TX: now also J10.2 (Pin_2)
- net ICM_EN: now reaches U6.123 (PG10)
- net ISM_EN: now reaches U6.48 (PC5)
- net CUR_SCL renamed I2C_SCL
- net I2C_SCL: now also J10.4 (Pin_4), J13.2 (Pin_2)
- net CUR_SDA renamed I2C_SDA
- net I2C_SDA: now also J10.5 (Pin_5), J13.3 (Pin_3)
- no-connect marks 49 -> 47
Other:
- note added: "I2C PIN HEADERS FOR AIR SPEED SENSOR (PITOT TUBE)"
- note added: "UART AND I2C CONNECTIONS"
- note added: "UART PIN HEADERS FOR GPS MODULE"
- note removed: "UART AND 5V CONNECTIONS"
- moved on the sheet: J11, J3, J5, J6, J7

Commit message: schematic changes
Parts:
- removed J1: Conn_01x06_Pin, Connector_PinHeader_2.54mm:PinHeader_1x06_P2.54mm_Vertical, symbol Connector:Conn_01x06_Pin
- added C53, C63: 100n, Capacitor_SMD:C_0805_2012Metric_Pad1.18x1.45mm_HandSolder, symbol Device:C
- added C64, C65: 4.7n, Capacitor_SMD:C_0805_2012Metric_Pad1.18x1.45mm_HandSolder, symbol Device:C
- added J14: Conn_01x05, Connector_PinHeader_2.54mm:PinHeader_1x05_P2.54mm_Vertical, symbol Connector_Generic:Conn_01x05
- added R22, R23, R34, R35: 60R, Resistor_SMD:R_0805_2012Metric_Pad1.20x1.40mm_HandSolder, symbol Device:R
Connections:
- net +3.3V: now also U7.5 (VIO), U8.5 (VIO), C53.1, C63.1, J14.5 (Pin_5)
- net CAN1H: now also R22.1
- net CAN1L: now also R23.2
- net CAN2H: now also R34.1
- net CAN2L: now also R35.2
- net GND: now also C53.2, C63.2, C64.1, C65.1, J14.1 (Pin_1)
- net NRST: now also J14.2 (Pin_2)
- net SWDCLK: now also J14.3 (Pin_3)
- net SWDIO: now also J14.4 (Pin_4)
- net JTDI: no longer names the net of U6.108 (PA15)
- net SWO: no longer names the net of U6.130 (PB3)
- new net: C64.2, R22.2, R23.1
- new net: C65.2, R34.2, R35.1
- no-connect marks 47 -> 49
Other:
- moved on the sheet: J2, J4

Commit message: power rails have been revised
Parts:
- removed J11, J3, J5, J6, J7: Conn_01x03_Pin, Connector_PinHeader_2.54mm:PinHeader_1x03_P2.54mm_Vertical, symbol Connector:Conn_01x03_Pin
- removed R15, R16, R17, R18: 33, Resistor_SMD:R_0805_2012Metric_Pad1.20x1.40mm_HandSolder, symbol Device:R
- added J1: Conn_01x04_Pin, Connector_JST:JST_GH_SM04B-GHS-TB_1x04-1MP_P1.25mm_Horizontal, symbol Connector:Conn_01x04_Pin
- added J3: Conn_01x06, Connector_JST:JST_GH_SM06B-GHS-TB_1x06-1MP_P1.25mm_Horizontal, symbol Connector_Generic:Conn_01x06
Connections:
- net +5V: now also J1.1 (Pin_1), J3.6 (Pin_6)
- net CAN2_RX: now also U6.72 (PB12); no longer U6.73 (PB13)
- net CAN2_TX: now also U6.73 (PB13); no longer U6.72 (PB12)
- net GND: now also J1.4 (Pin_4), J3.1 (Pin_1)
- net USART1_RX: now also J1.2 (Pin_2)
- net USART1_TX: now also J1.3 (Pin_3)
- net V_BAK: now reaches U6.28 (PC0)
- net V_BAK: now also J3.3 (Pin_3)
- net ST: now reaches U6.49 (PB0)
- net ST: now also J3.4 (Pin_4)
- net PGOOD_MAIN: now reaches U6.50 (PB1)
- net PGOOD_MAIN: now also J3.2 (Pin_2)
- net 5V_CRIT: now reaches U6.52 (PF11)
- net 5V_CRIT: now also J3.5 (Pin_5)
Other:
- note added: "Voltage Sensing"
- note removed: "PWM OUTPUTS (for revA)"
